Commit message: ADD: A - ABB_6700_with_track  B - Two robot setup

File: abb_irbt6004_670_support/urdf/abb_irb6700_175_305_ibois.xacro (robot description, xacro)
@@ -2,4 +2,10 @@
 <robot name="abb_irb6700_175_305_ibois" xmlns:xacro="http://ros.org/wiki/xacro">
   <xacro:include filename="$(find abb_irbt6004_670_support)/urdf/abb_irb6700_175_305_ibois_macro.xacro"/>
-  <xacro:abb_irb6700_175_305_ibois />
+  <link name="world" />
+  <joint name="world_joint" type="fixed">
+      <parent link="world" />
+      <child link = "rob1_axis" />
+      <origin xyz="0.0 0.0 0.0" rpy="0.0 0.0 0.0" />
+  </joint>
+  <xacro:abb_irb6700_175_305_ibois prefix="rob1_" />
 </robot>

File: abb_irbt6004_670_support/urdf/abb_irb6700_175_305_ibois_macro.xacro (robot description, xacro)
@@ -1,22 +1,17 @@
 <?xml version="1.0"?>
 <robot xmlns:xacro="http://wiki.ros.org/xacro">
-  <xacro:macro name="abb_irb6700_175_305_ibois">
-  <xacro:include filename="$(find abb_resources)/urdf/common_materials.xacro"/>
-  <xacro:include filename="$(find abb_irb6700_support)/urdf/irb6700_175_305_macro.xacro"/>
-  <xacro:include filename="$(find abb_irbt6004_670_support)/urdf/abb_irbt6004_670.xacro"/>
-  <link name="world" />
-  <joint name="world_joint" type="fixed">
-    <parent link="world" />
-    <child link = "axis" />
-    <origin xyz="0.0 0.0 0.0" rpy="0.0 0.0 0.0" />
-  </joint>
-  <xacro:abb_irbt6004_670 />
-  <joint name="abb_joint" type="fixed">
-    <parent link="pedestal"/>
-    <child  link="base_link"/>
-    <origin xyz="0 0 0 " rpy="0 0 0 "/>
-    <dynamics damping="0.2" friction="0" />
-  </joint>
-  <xacro:abb_irb6700_175_305 prefix=""/>
+  <xacro:macro name="abb_irb6700_175_305_ibois" params="prefix" >
+  <!--<xacro:macro name="abb_irb6700_175_305_ibois" params="prefix prefix_notused" >-->
+    <xacro:include filename="$(find abb_resources)/urdf/common_materials.xacro"/>
+    <xacro:include filename="$(find abb_irb6700_support)/urdf/irb6700_175_305_macro.xacro"/>
+    <xacro:include filename="$(find abb_irbt6004_670_support)/urdf/abb_irbt6004_670.xacro"/>
+    <xacro:abb_irbt6004_670 prefix="${prefix}" />
+    <joint name="${prefix}abb_joint" type="fixed">
+      <parent link="${prefix}pedestal"/>
+      <child  link="${prefix}base_link"/>
+      <origin xyz="0 0 0 " rpy="0 0 0 "/> <!--rotation of robot pedestal-->
+      <dynamics damping="0.2" friction="0" />
+    </joint>
+    <xacro:abb_irb6700_175_305 prefix="${prefix}"/><!--for multiple robots-->
   </xacro:macro>
 </robot>

File: abb_irbt6004_670_support/urdf/abb_irbt6004_670.xacro (robot description, xacro)
@@ -1,32 +1,33 @@
 <?xml version="1.0"?>
 <robot xmlns:xacro="http://wiki.ros.org/xacro">
-  <xacro:macro name="abb_irbt6004_670">
-    <link name="axis">
+  <xacro:macro name="abb_irbt6004_670" params="prefix">
+    <link name="${prefix}axis">
       <inertial>
-        <origin xyz="0.0 0.0 0.0"/>
         <mass value="120"/>
         <inertia ixx="-4.98000" iyy="-5.95200" izz="0.82800" ixy="-0.00000" ixz="2.70000" iyz="-0.00000"/>
       </inertial>
       <visual>
+        <origin xyz="3.35 0.0 0.0"/>
         <geometry>
-          <mesh filename="package://abb_irbt6004_670_support/abb_irbt6004_670/meshes/visual/axis.stl"/>
+          <mesh filename="package://abb_irbt6004_670_support/meshes/abb_irbt6004_670/visual/axis.stl"/>
         </geometry>
         <xacro:material_abb_white />
       </visual>
       <collision>
+        <origin xyz="3.35 0.0 0.0"/>
         <geometry>
-          <mesh filename="package://abb_irbt6004_670_support/abb_irbt6004_670/meshes/collision/axis.stl"/>
+          <mesh filename="package://abb_irbt6004_670_support/meshes/abb_irbt6004_670/collision/axis.stl"/>
         </geometry>
       </collision>
     </link>
-    <joint name="linear_axis_joint" type="prismatic">
-      <parent link="axis"/>
-      <child  link="pedestal"/>
-      <origin xyz="1.926 0.349 0.812" rpy="0 0 0 "/>
+    <joint name="${prefix}linear_axis_joint" type="prismatic">
+      <parent link="${prefix}axis"/>
+      <child  link="${prefix}pedestal"/>
+      <origin xyz="0 0 0.05" rpy="0 0 0 "/> <!--track origin or translation from origin-->
       <axis   xyz="1 0 0"/>
-      <limit lower="-1.926" upper="0.675" effort="100000" velocity="2.618" />
+      <limit lower="0" upper="6.700" effort="100000" velocity="2.618" />  <!--track limits or length-->
       <dynamics damping="0.2" friction="0" />
     </joint>
-    <link name="pedestal">
+    <link name="${prefix}pedestal">
       <inertial>
         <origin xyz="0.0 0.0 0.0"/>
@@ -36,5 +37,5 @@
       <visual>
         <geometry>
-          <mesh filename="package://abb_irbt6004_670_support/abb_irbt6004_670/meshes/visual/pedestal_250.stl"/>
+          <mesh filename="package://abb_irbt6004_670_support/meshes/abb_irbt6004_670/visual/pedestal_250.stl"/>
         </geometry>
         <xacro:material_abb_white />
@@ -42,5 +43,5 @@
       <collision>
         <geometry>
-          <mesh filename="package://abb_irbt6004_670_support/abb_irbt6004_670/meshes/collision/pedestal_250.stl"/>
+          <mesh filename="package://abb_irbt6004_670_support/meshes/abb_irbt6004_670/collision/pedestal_250.stl"/>
         </geometry>
       </collision>
